Commit message: added the test tube in the urdf and inside the launch

File: urdf/test_tube/test_tube.gazebo.xacro (robot description, xacro)
@@ -1,5 +1,5 @@
 <?xml version="1.0"?>
 <robot xmlns:xacro="http://www.ros.org/wiki/xacro">
-  <xacro:macro name="test_tube_gazebo" params="prefix"/>
+  <xacro:macro name="test_tube_gazebo" params="prefix">
     <gazebo reference="${prefix}tube_link">
       <static>false</static>

File: urdf/test_tube/test_tube.urdf.xacro (robot description, xacro)
@@ -6,8 +6,5 @@
         <origin xyz="0 0 0" rpy="0 0 0"/>
         <geometry>
-          <cylinder>
-            <radius>0.0180</radius>
-            <length>0.1030</length>
-          </cylinder>
+          <cylinder radius="0.0180" length="0.1030"/>
         </geometry>
       </visual>
@@ -15,8 +12,5 @@
         <origin xyz="0 0 0" rpy="0 0 0"/>
         <geometry>
-          <cylinder>
-            <radius>0.0180</radius>
-            <length>0.1030</length>
-          </cylinder>
+          <cylinder radius="0.0180" length="0.1030"/>
         </geometry>
       </collision>

File: urdf/test_tube/test_tube.xacro (robot description, xacro)
@@ -3,8 +3,8 @@
   <xacro:arg name="prefix" default="test_tube_1_"/>
   <!-- Includo URDF e argomento -->
-  <xacro:include filename="$(find YumiProjectThesis)/urdf/test_tube.urdf.xacro"/>
+  <xacro:include filename="$(find YumiProjectThesis)/urdf/test_tube/test_tube.urdf.xacro"/>
   <xacro:test_tube_urdf prefix="$(arg prefix)"/>
   <!-- Gazebo -->
-  <xacro:include filename="$(find YumiProjectThesis)/urdf/test_tube.gazebo.xacro"/>
+  <xacro:include filename="$(find YumiProjectThesis)/urdf/test_tube/test_tube.gazebo.xacro"/>
   <xacro:test_tube_gazebo prefix="$(arg prefix)"/>
 </robot>
